Commit message: Recreated pi_robot.urdf using xacro

File: rbx2_description/urdf/pi_robot/pi_robot.urdf (robot description, URDF)
Before this commit: robot pi_robot, 40 links, 39 joints
Joints:
- joint right_arm_shoulder_pan_joint: limit lower=-1.57 upper=1.57 effort=1.0 velocity=3.14 -> lower=-2.09 upper=2.09 effort=1.0 velocity=3.14
