Commit message: Shifted origin of Xtion Pro STL model 2 cm to place origin in the middle of the camera

File: rbx2_description/urdf/pi_robot/pi_pan_tilt_head_xtion.urdf.xacro (robot description, xacro)
@@ -3,5 +3,5 @@
   <property name="camera_offset_x" value="0.0" />
   <property name="camera_offset_y" value="0.0" />
-  <property name="camera_offset_z" value="0.04" />
+  <property name="camera_offset_z" value="0.06" />
   <property name="camera_mesh_scale" value="1.0" />
   <xacro:include filename="$(find rbx2_description)/urdf/pi_robot/dynamixel_head_hardware.xacro" />

File: rbx2_description/urdf/pi_robot/pi_robot_with_xtion.xacro (robot description, xacro)
@@ -7,5 +7,5 @@
    <property name="camera_offset_x" value="0.009" />
    <property name="camera_offset_y" value="0.0045" />
-   <property name="camera_offset_z" value="0.897" />
+   <property name="camera_offset_z" value="0.917" />
    <!-- The following include files set up definitions of parts of the robot body -->
    <xacro:include filename="$(find rbx2_description)/urdf/materials.urdf.xacro" />

File: rbx2_description/urdf/pi_robot/xtion.urdf.xacro (robot description, xacro)
@@ -16,5 +16,5 @@
       <link name="${name}_link">
          <visual>
-            <origin xyz="0 0 0" rpy="0 0 0"/>
+            <origin xyz="0 0 -0.02" rpy="0 0 0"/>
             <geometry>
                <mesh filename="package://rbx2_description/meshes/xtion.stl" scale="${camera_mesh_scale} ${camera_mesh_scale} ${camera_mesh_scale}" />
